File: Teensy perfboard/teensy perf schematic_2.sch (EAGLE design)
At the start: 16 parts

Commit message: More complete perfboard
Parts:
- removed JP1/BAR30, TEMP/HUM_HEADER: (no value), pinhead:PINHD-2X2
- added J1: Bar30, SparkFun-Connectors:M04PTH
- added J2: Temp/Hum, SparkFun-Connectors:M04PTH
- added J3: LED, SparkFun-Connectors:M04PTH
- added SG1: BUZZERPTH, SparkFun-Electromechanical:BUZZERPTH
Connections:
- removed net N$20 (its old number): SENSOR.3.3V, TEMP/HUM_HEADER.3
- removed net N$22: TEMP/HUM_HEADER.2
- new net +3V3: J1.4
- new net +5V: J2.4, SENSOR.VIN
- new net N$1: J1.2, SENSOR.19/A5/T/SCL0
- new net N$11: J2.1, SENSOR.15/A1/T
- new net N$12: GPIO.GND, POWER.GND, THRUSTER.GND
- new net N$13: GPIO.20/A6/PWM, SG1.2
- new net N$9: THRUSTER.21/A7/PWM
- net GND: now also J1.1, J2.3, SENSOR.AGND, SG1.1; no longer GPIO.GND, POWER.GND, TEMP/HUM_HEADER.4, THRUSTER.GND
- net N$10: now also J1.3, SENSOR.18/A4/T/SDA0; no longer JP1/BAR30.4
- net N$2: now also THRUSTER.3/CAN-TX/PWM
- net N$21: now also J2.2, SENSOR.14/A0; no longer TEMP/HUM_HEADER.1
- net N$3: now also THRUSTER.4/CAN-RX-PWM
- net N$4: now also THRUSTER.5/PWM
- net N$5: now also THRUSTER.6/PWM
- net N$6: now also THRUSTER.9/RX2/PWM
- net N$7: now also THRUSTER.10/TX2/PWM
- net N$8: now also THRUSTER.20/A6/PWM
Other:
- moved on the sheet: ESC1, ESC2, ESC3, ESC4, SENSOR
